File: macro_pad.kicad_pcb (KiCad board)
At the start: 2 copper layers, 112.3 x 92.7 mm, 53 parts, among them J1 OLED, J2 SWD, SW1 SW_Push_45deg, SW10 SW_Push_45deg, SW11 SW_Push_45deg, SW12 SW_Push_45deg, SW13 SW_Push_45deg, SW14 SW_Push_45deg, SW15 SW_Push_45deg, SW16 SW_Push_45deg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

Commit message: Added mounting holes
Parts:
- added H1: MountingHole, MountingHole:MountingHole_3.2mm_M3, F.Cu at (127.8, 113.4)
- added H2: MountingHole, MountingHole:MountingHole_3.2mm_M3, F.Cu at (128.1, 75.3)
- added H3: MountingHole, MountingHole:MountingHole_3.2mm_M3, F.Cu at (70.9, 75.3)
- added H4: MountingHole, MountingHole:MountingHole_3.2mm_M3, F.Cu at (70.9, 113.4)
- R1: moved to B.Cu
- moved R1 7.00 mm to (131.6, 89.5)
- moved R2 1.69 mm to (77.0, 44.8)
Routing:
- net Net-(D17-DIN): track 12.6 -> 21.3 mm
- net /LedData: track 30.8 -> 27.8 mm
- net Net-(D19-DOUT): track 14.5 -> 17.0 mm
- net Net-(D27-DOUT): track 14.5 -> 16.4 mm
- net /BrEncB: track 71.0 -> 72.2 mm
- net /BrEncA: track 72.5 -> 73.4 mm
